File: PCBs/CNC_Control_Panel/CNC_Control_Panel.kicad_pcb (KiCad board)
At the start: 2 copper layers, 20 parts, among them J1 Raspberry_Pi_2_3

Commit message: Cleanup
Parts:
- removed D_OnOff1: SFH4346, LED_THT:LED_D3.0mm_IRBlack
- removed R2, R3, R4, R5, R6, R7, R8, R9: 100k, Resistor_THT:R_Axial_DIN0207_L6.3mm_D2.5mm_P7.62mm_Horizontal
- removed SW_$H_Home1, SW_$X_Unlock1, SW_Left1, SW_OnOffButton1, SW_Right1, SW_Y_Down1, SW_Y_Up1, SW_Z_Down1, SW_Z_Up1: SW_Push_Dual, Button_Switch_THT:SW_PUSH_6mm
- added $H_HOME1: SW_Push_Dual, Button_Switch_THT:SW_PUSH_6mm, F.Cu at (79.0, 146.3)
- added $X_UNLOCK1: SW_Push_Dual, Button_Switch_THT:SW_PUSH_6mm, F.Cu at (85.2, 127.3)
- added C-CTRL_RESET1: SW_Push_Dual, Button_Switch_THT:SW_PUSH_6mm, F.Cu at (94.8, 127.3)
- added J2: Conn_01x07_Male, Connector_PinSocket_2.54mm:PinSocket_1x07_P2.54mm_Vertical_SMD_Pin1Left, F.Cu at (80.6, 135.3)
- added ON_OFF-LED1: RedLED3mm, LED_THT:LED_D5.0mm, F.Cu at (108.1, 144.1)
- added ON_OFF1: SW_Push_Dual, Button_Switch_THT:SW_PUSH_6mm, F.Cu at (104.3, 127.3)
- added PAUSE_RESUME1: SW_Push_Dual, Button_Switch_THT:SW_PUSH_6mm, F.Cu at (85.2, 134.8)
- added X-DECR1: SW_Push_Dual, Button_Switch_THT:SW_PUSH_6mm, F.Cu at (94.8, 134.8)
- added X-INCR1: SW_Push_Dual, Button_Switch_THT:SW_PUSH_6mm, F.Cu at (88.5, 142.4)
- added X-ZERO1: SW_Push_Dual, Button_Switch_THT:SW_PUSH_6mm, F.Cu at (104.3, 134.8)
- added Y-DECR1: SW_Push_Dual, Button_Switch_THT:SW_PUSH_6mm, F.Cu at (88.5, 149.9)
- added Y-INCR1: SW_Push_Dual, Button_Switch_THT:SW_PUSH_6mm, F.Cu at (113.9, 127.3)
- added Y-ZERO1: SW_Push_Dual, Button_Switch_THT:SW_PUSH_6mm, F.Cu at (98.1, 142.4)
- added Z-DECR1: SW_Push_Dual, Button_Switch_THT:SW_PUSH_6mm, F.Cu at (113.9, 134.8)
- added Z-INCR1: SW_Push_Dual, Button_Switch_THT:SW_PUSH_6mm, F.Cu at (98.1, 149.9)
- added Z-ZERO1: SW_Push_Dual, Button_Switch_THT:SW_PUSH_6mm, F.Cu at (123.4, 127.3)
- R1: value 100k -> 1k
Connections:
- J1 pad 11: Net-(J1-Pad11) -> Y0
- J1 pad 12: Net-(J1-Pad12) -> Z0
- J1 pad 14: Net-(J1-Pad14) -> GND
- J1 pad 19: Net-(J1-Pad19) -> ON_OFF
- J1 pad 20: Net-(J1-Pad20) -> GND
- J1 pad 21: Net-(J1-Pad21) -> Z-INCR
- J1 pad 23: Net-(J1-Pad23) -> HOME
- J1 pad 24: Net-(J1-Pad24) -> Z-DECR
- J1 pad 25: Net-(J1-Pad25) -> GND
- J1 pad 26: Net-(J1-Pad26) -> Y-INCR
- J1 pad 29: Net-(J1-Pad29) -> X-INCR
- J1 pad 30: Net-(J1-Pad30) -> GND
- J1 pad 31: Net-(J1-Pad31) -> Y-DECR
- J1 pad 32: Net-(J1-Pad32) -> UNLOCK
- J1 pad 33: Net-(J1-Pad33) -> RESET
- J1 pad 34: Net-(J1-Pad34) -> GND
- J1 pad 35: Net-(J1-Pad35) -> PAUSE
- J1 pad 36: Net-(J1-Pad36) -> X0
- J1 pad 39: Net-(D_OnOff1-Pad1) -> GND
- J1 pad 6: Net-(J1-Pad6) -> GND
- J1 pad 7: Net-(J1-Pad7) -> X-DECR
- J1 pad 9: Net-(J1-Pad9) -> GND
- R1 pad 1: Net-(J1-Pad1) -> GND
- R1 pad 2: Net-(J1-Pad7) -> Net-(ON_OFF-LED1-Pad1)
Routing:
- net Net-(D_OnOff1-Pad1): track 211.8 -> 0.00 mm
- net Net-(J1-Pad7): track 98.3 -> 0.00 mm
- net Net-(J1-Pad23): track 81.6 -> 0.00 mm
- net Net-(J1-Pad8): track 80.6 -> 0.00 mm
- net Net-(J1-Pad29): track 76.7 -> 0.00 mm
- net Net-(J1-Pad32): track 76.3 -> 0.00 mm
- net Net-(J1-Pad21): track 70.4 -> 0.00 mm
- net Net-(J1-Pad1): track 66.1 -> 0.00 mm
- net Net-(J1-Pad19): track 63.8 -> 0.00 mm
- net Net-(J1-Pad24): track 61.1 -> 0.00 mm
- net Net-(J1-Pad26): track 56.3 -> 0.00 mm
- net Net-(J1-Pad27): track 55.8 -> 0.00 mm
