File: PCBs/CNC_Control_Panel/CNC_Control_Panel.kicad_pcb (KiCad board)
At the start: 2 copper layers, 100 x 100 mm, 50 parts, among them J1 Conn_01x07_Male, J2 Conn_01x03_Male, J3 Conn_01x07_Male, P1 Conn_02x20_Odd_Even, Q1 BSS138, X0 SW_Push, Y0 SW_Push

Commit message: generated Gerber files
Other:
- board text added: "by Pakue (2018)"
Changed lines of the file:
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@@
   (general
     (thickness 1.6)
-    (drawings 49)
+    (drawings 59)
     (tracks 400)
     (zones 0)
@@
     (pad_to_mask_clearance 0)
     (aux_axis_origin 36.636 85.745)
-    (grid_origin 36.636 85.745)
+    (grid_origin 134.272 80.478)
     (visible_elements 7FFFFFFF)
     (pcbplotparams
-      (layerselection 0x00030_80000001)
+      (layerselection 0x010f0_ffffffff)
       (usegerberextensions true)
-      (usegerberattributes false)
+      (usegerberattributes true)
       (usegerberadvancedattributes false)
       (creategerberjobfile false)
@@
       (outputformat 1)
       (mirror false)
-      (drillshape 1)
+      (drillshape 0)
       (scaleselection 1)
-      (outputdirectory ""))
+      (outputdirectory "gerbers/"))
   )
   (net 0 "")
@@
     )
   )
+  (dimension 11 (width 0.25) (layer Dwgs.User)
+    (gr_text "11.000 mm" (at 128.772 89.978) (layer Dwgs.User)
+      (effects (font (size 1 1) (thickness 0.25)))
+    )
+    (feature1 (pts (xy 134.272 88.478) (xy 134.272 89.064421)))
+    (feature2 (pts (xy 123.272 88.478) (xy 123.272 89.064421)))
+    (crossbar (pts (xy 123.272 88.478) (xy 134.272 88.478)))
+    (arrow1a (pts (xy 134.272 88.478) (xy 133.145496 89.064421)))
+    (arrow1b (pts (xy 134.272 88.478) (xy 133.145496 87.891579)))
+    (arrow2a (pts (xy 123.272 88.478) (xy 124.398504 89.064421)))
+    (arrow2b (pts (xy 123.272 88.478) (xy 124.398504 87.891579)))
+  )
+  (dimension 30 (width 0.25) (layer Dwgs.User)
+    (gr_text "30.000 mm" (at 110.772 114.978 90) (layer Dwgs.User)
+      (effects (font (size 1 1) (thickness 0.25)))
+    )
+    (feature1 (pts (xy 98.272 99.978) (xy 109.858421 99.978)))
+    (feature2 (pts (xy 98.272 129.978) (xy 109.858421 129.978)))
+    (crossbar (pts (xy 109.272 129.978) (xy 109.272 99.978)))
+    (arrow1a (pts (xy 109.272 99.978) (xy 109.858421 101.104504)))
+    (arrow1b (pts (xy 109.272 99.978) (xy 108.685579 101.104504)))
+    (arrow2a (pts (xy 109.272 129.978) (xy 109.858421 128.851496)))
+    (arrow2b (pts (xy 109.272 129.978) (xy 108.685579 128.851496)))
+  )
+  (dimension 40 (width 0.25) (layer Dwgs.User)
+    (gr_text "40.000 mm" (at 75.772 114.978 270) (layer Dwgs.User)
+      (effects (font (size 1 1) (thickness 0.25)))
+    )
+    (feature1 (pts (xy 63.272 134.978) (xy 74.858421 134.978)))
+    (feature2 (pts (xy 63.272 94.978) (xy 74.858421 94.978)))
+    (crossbar (pts (xy 74.272 94.978) (xy 74.272 134.978)))
+    (arrow1a (pts (xy 74.272 134.978) (xy 73.685579 133.851496)))
+    (arrow1b (pts (xy 74.272 134.978) (xy 74.858421 133.851496)))
+    (arrow2a (pts (xy 74.272 94.978) (xy 73.685579 96.104504)))
+    (arrow2b (pts (xy 74.272 94.978) (xy 74.858421 96.104504)))
+  )
+  (dimension 40 (width 0.25) (layer Dwgs.User)
+    (gr_text "40.000 mm" (at 63.272 118.477999) (layer Dwgs.User)
+      (effects (font (size 1 1) (thickness 0.25)))
+    )
+    (feature1 (pts (xy 83.272 114.978) (xy 83.272 117.56442)))
+    (feature2 (pts (xy 43.272 114.978) (xy 43.272 117.56442)))
+    (crossbar (pts (xy 43.272 116.977999) (xy 83.272 116.977999)))
+    (arrow1a (pts (xy 83.272 116.977999) (xy 82.145496 117.56442)))
+    (arrow1b (pts (xy 83.272 116.977999) (xy 82.145496 116.391578)))
+    (arrow2a (pts (xy 43.272 116.977999) (xy 44.398504 117.56442)))
+    (arrow2b (pts (xy 43.272 116.977999) (xy 44.398504 116.391578)))
+  )
+  (dimension 15 (width 0.25) (layer Dwgs.User)
+    (gr_text "15.000 mm" (at 131.772 137.478 90) (layer Dwgs.User)
+      (effects (font (size 1 1) (thickness 0.25)))
+    )
+    (feature1 (pts (xy 120.272 129.978) (xy 130.858421 129.978)))
+    (feature2 (pts (xy 120.272 144.978) (xy 130.858421 144.978)))
+    (crossbar (pts (xy 130.272 144.978) (xy 130.272 129.978)))
+    (arrow1a (pts (xy 130.272 129.978) (xy 130.858421 131.104504)))
+    (arrow1b (pts (xy 130.272 129.978) (xy 129.685579 131.104504)))
+    (arrow2a (pts (xy 130.272 144.978) (xy 130.858421 143.851496)))
+    (arrow2b (pts (xy 130.272 144.978) (xy 129.685579 143.851496)))
+  )
+  (dimension 20 (width 0.25) (layer Dwgs.User)
+    (gr_text "20.000 mm" (at 131.772 154.978 90) (layer Dwgs.User)
+      (effects (font (size 1 1) (thickness 0.25)))
+    )
+    (feature1 (pts (xy 120.272 144.978) (xy 130.858421 144.978)))
+    (feature2 (pts (xy 120.272 164.978) (xy 130.858421 164.978)))
+    (crossbar (pts (xy 130.272 164.978) (xy 130.272 144.978)))
+    (arrow1a (pts (xy 130.272 144.978) (xy 130.858421 146.104504)))
+    (arrow1b (pts (xy 130.272 144.978) (xy 129.685579 146.104504)))
+    (arrow2a (pts (xy 130.272 164.978) (xy 130.858421 163.851496)))
+    (arrow2b (pts (xy 130.272 164.978) (xy 129.685579 163.851496)))
+  )
+  (dimension 20 (width 0.25) (layer Dwgs.User)
+    (gr_text "20.000 mm" (at 70.272 169.478) (layer Dwgs.User)
+      (effects (font (size 1 1) (thickness 0.25)))
+    )
+    (feature1 (pts (xy 80.272 164.978) (xy 80.272 168.564421)))
+    (feature2 (pts (xy 60.272 164.978) (xy 60.272 168.564421)))
+    (crossbar (pts (xy 60.272 167.978) (xy 80.272 167.978)))
+    (arrow1a (pts (xy 80.272 167.978) (xy 79.145496 168.564421)))
+    (arrow1b (pts (xy 80.272 167.978) (xy 79.145496 167.391579)))
+    (arrow2a (pts (xy 60.272 167.978) (xy 61.398504 168.564421)))
+    (arrow2b (pts (xy 60.272 167.978) (xy 61.398504 167.391579)))
+  )
+  (dimension 70 (width 0.25) (layer Dwgs.User)
+    (gr_text "70.000 mm" (at 138.772 136.478 90) (layer Dwgs.User)
+      (effects (font (size 1 1) (thickness 0.25)))
+    )
+    (feature1 (pts (xy 128.272 101.478) (xy 137.858421 101.478)))
+    (feature2 (pts (xy 128.272 171.478) (xy 137.858421 171.478)))
+    (crossbar (pts (xy 137.272 171.478) (xy 137.272 101.478)))
+    (arrow1a (pts (xy 137.272 101.478) (xy 137.858421 102.604504)))
+    (arrow1b (pts (xy 137.272 101.478) (xy 136.685579 102.604504)))
+    (arrow2a (pts (xy 137.272 171.478) (xy 137.858421 170.351496)))
+    (arrow2b (pts (xy 137.272 171.478) (xy 136.685579 170.351496)))
+  )
+  (dimension 88 (width 0.25) (layer Dwgs.User)
+    (gr_text "88.000 mm" (at 84.272 181.977999) (layer Dwgs.User)
+      (effects (font (size 1 1) (thickness 0.25)))
+    )
+    (feature1 (pts (xy 128.272 171.478) (xy 128.272 181.06442)))
+    (feature2 (pts (xy 40.272 171.478) (xy 40.272 181.06442)))
+    (crossbar (pts (xy 40.272 180.477999) (xy 128.272 180.477999)))
+    (arrow1a (pts (xy 128.272 180.477999) (xy 127.145496 181.06442)))
+    (arrow1b (pts (xy 128.272 180.477999) (xy 127.145496 179.891578)))
+    (arrow2a (pts (xy 40.272 180.477999) (xy 41.398504 181.06442)))
+    (arrow2b (pts (xy 40.272 180.477999) (xy 41.398504 179.891578)))
+  )
+  (gr_text "by Pakue (2018)" (at 110.804 175.407) (layer F.SilkS)
+    (effects (font (size 1 1) (thickness 0.25)))
+  )
   (gr_text 5V (at 55.94 154.579) (layer B.SilkS)
