File: PCBs/CNC_Control_Panel/CNC_Control_Panel.sch (KiCad schematic (older format))
At the start: 20 parts, among them J1 Raspberry_Pi_2_3

Commit message: started cleaning up the schematic and added new functions
Parts:
- removed R1, R2, R3, R4, R5, R6, R7, R8, R9: 100k, Resistor_THT:R_Axial_DIN0207_L6.3mm_D2.5mm_P7.62mm_Horizontal, symbol Device:R
- removed SW_$H_Home1, SW_$X_Unlock1, SW_Left1, SW_OnOffButton1, SW_Right1, SW_Y_Down1, SW_Y_Up1, SW_Z_Down1, SW_Z_Up1: SW_Push_Dual, Button_Switch_THT:SW_PUSH_6mm, symbol Switch:SW_Push
- added $H_HOME, $X_UNLOCK, C-CTRL_RESET, ON_OFF, PAUSE_RESUME, X-DECR, X-INCR, X-ZERO, Y-DECR, Y-INCR, Y-ZERO, Z-DECR, Z-INCR, Z-ZERO: SW_Push_Dual, Button_Switch_THT:SW_PUSH_6mm, symbol Switch:SW_Push
- added J?: Conn_01x07_Male, symbol Connector:Conn_01x07_Male
- added R?: 1k, Resistor_THT:R_Axial_DIN0207_L6.3mm_D2.5mm_P7.62mm_Horizontal, symbol Device:R
- ON_OFF-LED: renamed from D_OnOff1; value SFH4346 -> RedLED3mm
Connections:
- net labels added: GND, HOME, ON_OFF, PAUSE, RESET, UNLOCK, X-DECR, X-INCR, X0, Y-DECR, Y-INCR, Y0, Z-DECR, Z-INCR, Z0
- wire segments 76 -> 28
Other:
- note added: "6x Rotation Switch\nRemember appropriate \ncutout on PCB"
- note added: "Additional bottons"
- note added: "Directional control"
- note added: "The GPIOs of the Raspi can have\nsoftware defined pullups, therefore\nno external ones are needed.\nSoftware implementation needed!"
- moved on the sheet: ON_OFF-LED

Commit message: Cleanup
Parts:
- J2: renamed from J?; footprint (none) -> Connector_PinSocket_2.54mm:PinSocket_1x07_P2.54mm_Vertical_SMD_Pin1Left
- ON_OFF-LED1: renamed from ON_OFF-LED; footprint LED_THT:LED_D3.0mm_IRBlack -> LED_THT:LED_D5.0mm
- gave numbers to parts that had none: 1
- renumbered $H_HOME to $H_HOME1, $X_UNLOCK to $X_UNLOCK1, C-CTRL_RESET to C-CTRL_RESET1, ON_OFF to ON_OFF1, PAUSE_RESUME to PAUSE_RESUME1, X-DECR to X-DECR1, X-INCR to X-INCR1, X-ZERO to X-ZERO1, Y-DECR to Y-DECR1, Y-INCR to Y-INCR1, Y-ZERO to Y-ZERO1, Z-DECR to Z-DECR1, Z-INCR to Z-INCR1, Z-ZERO to Z-ZERO1
Connections:
- no-connect marks 0 -> 11
