File: PCBs/CNC_Control_Panel/CNC_Control_Panel.sch (KiCad schematic (older format))
At the start: 20 parts, among them P1 Conn_02x20_Odd_Even, X0 SW_Push, Y0 SW_Push

Commit message: finished schematic and initial layout
Parts:
- added J1: Conn_01x07_Male, Connector_PinHeader_2.54mm:PinHeader_1x07_P2.54mm_Horizontal, symbol Connector:Conn_01x07_Male
- added ON_OFF1: SW_Push, Button_Switch_THT:SW_PUSH_6mm, symbol Switch:SW_Push
- $H_HOME1: renamed from $H_HOME; footprint (none) -> Button_Switch_THT:SW_PUSH_6mm
- $X_UNLOCK1: renamed from $X_UNLOCK; footprint (none) -> Button_Switch_THT:SW_PUSH_6mm
- C-CTRL_RESET1: renamed from C-CTRL_RESET; footprint (none) -> Button_Switch_THT:SW_PUSH_6mm
- D1: renamed from D?; footprint (none) -> LED_THT:LED_D5.0mm
- PAUSE_RESUME1: renamed from PAUSE_RESUME; footprint (none) -> Button_Switch_THT:SW_PUSH_6mm
- R1: renamed from R?; footprint (none) -> Resistor_THT:R_Axial_DIN0207_L6.3mm_D2.5mm_P7.62mm_Horizontal
- X-DECR1: renamed from X-DECR; footprint (none) -> Button_Switch_THT:SW_PUSH_6mm
- X-INCR1: renamed from X-INCR; footprint (none) -> Button_Switch_THT:SW_PUSH_6mm
- X0, Y0, Z0: footprint (none) -> Button_Switch_THT:SW_PUSH_6mm
- Y-DECR1, Z-DECR1: renamed from Y-DECR; footprint (none) -> Button_Switch_THT:SW_PUSH_6mm
- Y-INCR1, Z-INCR1: renamed from Y-INCR; footprint (none) -> Button_Switch_THT:SW_PUSH_6mm
Connections:
- wire segments 56 -> 78
Other:
- note added: "Directional Control"
- note added: "Functiomn Buttons"
- note added: "LED Indicator"
- note added: "Rotatry Switch"

Commit message: added external pullup resistors
Parts:
- added R? (x20): 10k, symbol Device:R
- R1: value R -> 470Ohm
Connections:
- wire segments 78 -> 129
Other:
- note added: "Function Buttons"
- note removed: "Functiomn Buttons"
- note removed: "Raspi GPIOs have internal pullup/-downs\nthat can be defined via software. Therfore \nno resistors should be needed for the input\nbuttons."

Commit message: new layout with a 100x100mm board design and cutout for a 8mm rotatary switch
Parts:
- R1: value 470Ohm -> 470; footprint Resistor_THT:R_Axial_DIN0207_L6.3mm_D2.5mm_P7.62mm_Horizontal -> Resistor_SMD:R_0805_2012Metric_Pad1.15x1.40mm_HandSolder
- R10, R11, R12, R13, R14, R15, R16, R17, R18, R19, R2, R20, R21, R3, R4, R5, R6, R7, R8, R9: renamed from R?; footprint (none) -> Resistor_SMD:R_0805_2012Metric_Pad1.15x1.40mm_HandSolder

Commit message: replaced the normal LED with a header for NeoPixels
Parts:
- removed D1: LED, LED_THT:LED_D5.0mm, symbol Device:LED
- removed R1: 470, Resistor_SMD:R_0805_2012Metric_Pad1.15x1.40mm_HandSolder, symbol Device:R
- added J2: Conn_01x03_Male, Connector_PinHeader_2.54mm:PinHeader_1x03_P2.54mm_Horizontal, symbol Connector:Conn_01x03_Male
- added Q?: BSS138, Package_TO_SOT_SMD:SOT-23, symbol Transistor_FET:BSS138
- added R? (x2): 10k, Resistor_SMD:R_0805_2012Metric_Pad1.15x1.40mm_HandSolder, symbol Device:R
Connections:
- wire segments 129 -> 142
Other:
- note added: "LED Indicator (WS2812B)"
- note removed: "LED Indicator"
Changed lines of the file:
@@
 $EndComp
-$Comp
-L Device:LED D1
-U 1 1 5BB2B2C5
-P 5800 1400
-F 0 "D1" V 5838 1283 50  0000 R CNN
-F 1 "LED" V 5747 1283 50  0000 R CNN
-F 2 "LED_THT:LED_D5.0mm" H 5800 1400 50  0001 C CNN
-F 3 "~" H 5800 1400 50  0001 C CNN
-	1    5800 1400
-	0    -1   -1   0
-$EndComp
-$Comp
-L Device:R R1
-U 1 1 5BB2B3BA
-P 5800 1800
-F 0 "R1" H 5870 1846 50  0000 L CNN
-F 1 "470" H 5870 1755 50  0000 L CNN
-F 2 "Resistor_SMD:R_0805_2012Metric_Pad1.15x1.40mm_HandSolder" V 5730 1800 50  0001 C CNN
-F 3 "~" H 5800 1800 50  0001 C CNN
-	1    5800 1800
-	1    0    0    -1
-$EndComp
-Wire Wire Line
-	5800 1250 5800 1100
-Wire Wire Line
-	5800 1650 5800 1550
-Wire Wire Line
-	5800 1950 5800 2100
-Wire Wire Line
-	5800 1100 5200 1100
 $Comp
 L Switch:SW_Push ON_OFF1
@@
 $EndComp
 $Comp
-L power:GND #PWR0101
-U 1 1 5BB26B90
-P 5800 2100
-F 0 "#PWR0101" H 5800 1850 50  0001 C CNN
-F 1 "GND" H 5805 1927 50  0000 C CNN
-F 2 "" H 5800 2100 50  0001 C CNN
-F 3 "" H 5800 2100 50  0001 C CNN
-	1    5800 2100
-	1    0    0    -1
-$EndComp
-$Comp
 L power:GND #PWR0102
 U 1 1 5BB26C81
@@
 Wire Wire Line
 	8150 5750 9000 5750
-Text Label 5200 1100 0    50   ~ 0
+Text Label 4350 1600 0    50   ~ 0
 GPIO12(PWM0)
 Text Label 1050 4500 0    50   ~ 0
@@
 	6700 2450 6700 800
 Wire Notes Line
-	5050 800  6250 800
-Wire Notes Line
-	6250 800  6250 2450
-Wire Notes Line
-	6250 2450 5050 2450
-Wire Notes Line
-	5050 2450 5050 800
+	4300 800  6600 800
+Wire Notes Line
+	6600 800  6600 2450
+Wire Notes Line
+	6600 2450 4300 2450
+Wire Notes Line
+	4300 2450 4300 800
 Wire Notes Line
 	5050 2650 10050 2650
@@
 Text Notes 950  3700 0    50   ~ 0
 Function Buttons
-Text Notes 5050 800  0    50   ~ 0
-LED Indicator
+Text Notes 4300 800  0    50   ~ 0
+LED Indicator (WS2812B)
 Text Notes 6700 800  0    50   ~ 0
 Rotatry Switch
@@
 	1    0    0    -1
 $EndComp
+$Comp
+L power:GND #PWR0101
+U 1 1 5BB26B90
+P 5800 1900
+F 0 "#PWR0101" H 5800 1650 50  0001 C CNN
+F 1 "GND" H 5805 1727 50  0000 C CNN
+F 2 "" H 5800 1900 50  0001 C CNN
+F 3 "" H 5800 1900 50  0001 C CNN
+	1    5800 1900
+	1    0    0    -1
+$EndComp
+$Comp
+L Connector:Conn_01x03_Male J2
+U 1 1 5BBAAFC2
+P 6100 1600
+F 0 "J2" H 6250 1350 50  0000 R CNN
+F 1 "Conn_01x03_Male" H 6350 1800 50  0000 R CNN
+F 2 "Connector_PinHeader_2.54mm:PinHeader_1x03_P2.54mm_Horizontal" H 6100 1600 50  0001 C CNN
+F 3 "~" H 6100 1600 50  0001 C CNN
+	1    6100 1600
+	-1   0    0    1
+$EndComp
+$Comp
+L power:+5V #PWR0126
+U 1 1 5BBAFD4B
+P 5800 1150
+F 0 "#PWR0126" H 5800 1000 50  0001 C CNN
+F 1 "+5V" H 5800 1290 50  0000 C CNN
+F 2 "" H 5800 1150 50  0000 C CNN
+F 3 "" H 5800 1150 50  0000 C CNN
+	1    5800 1150
+	1    0    0    -1
+$EndComp
+Wire Wire Line
+	5800 1900 5800 1700
+Wire Wire Line
+	5800 1700 5900 1700
+Wire Wire Line
+	5900 1500 5800 1500
+Wire Wire Line
+	5800 1500 5800 1200
+$Comp
+L Transistor_FET:BSS138 Q?
+U 1 1 5BBD252E
+P 5300 1500
+F 0 "Q?" V 5550 1500 50  0000 C CNN
+F 1 "BSS138" V 5641 1500 50  0000 C CNN
+F 2 "Package_TO_SOT_SMD:SOT-23" H 5500 1425 50  0001 L CIN
+F 3 "https://www.fairchildsemi.com/datasheets/BS/BSS138.pdf" H 5300 1500 50  0001 L CNN
+	1    5300 1500
+	0    1    1    0
+$EndComp
+$Comp
+L Device:R R?
+U 1 1 5BC07184
+P 5550 1400
+F 0 "R?" H 5620 1446 50  0000 L CNN
+F 1 "10k" H 5620 1355 50  0000 L CNN
+F 2 "Resistor_SMD:R_0805_2012Metric_Pad1.15x1.40mm_HandSolder" V 5480 1400 50  0001 C CNN
+F 3 "~" H 5550 1400 50  0001 C CNN
+	1    5550 1400
+	1    0    0    -1
+$EndComp
+Wire Wire Line
+	5550 1250 5550 1200
+Wire Wire Line
+	5550 1200 5800 1200
+Connection ~ 5800 1200
+Wire Wire Line
+	5800 1200 5800 1150
+Wire Wire Line
+	5550 1550 5550 1600
+Wire Wire Line
+	5550 1600 5500 1600
+Wire Wire Line
+	5550 1600 5900 1600
+Connection ~ 5550 1600
+Wire Wire Line
+	5100 1600 5000 1600
+$Comp
+L Device:R R?
+U 1 1 5BC3AC59
+P 5000 1400
+F 0 "R?" H 5070 1446 50  0000 L CNN
+F 1 "10k" H 5070 1355 50  0000 L CNN
+F 2 "Resistor_SMD:R_0805_2012Metric_Pad1.15x1.40mm_HandSolder" V 4930 1400 50  0001 C CNN
+F 3 "~" H 5000 1400 50  0001 C CNN
+	1    5000 1400
+	1    0    0    -1
+$EndComp
+$Comp
+L power:+3.3V #PWR?
+U 1 1 5BC3ADA5
+P 5000 1150
+F 0 "#PWR?" H 5000 1000 50  0001 C CNN
+F 1 "+3.3V" H 5000 1290 50  0000 C CNN
+F 2 "" H 5000 1150 50  0000 C CNN
+F 3 "" H 5000 1150 50  0000 C CNN
+	1    5000 1150
+	1    0    0    -1
+$EndComp
+Wire Wire Line
+	5000 1250 5000 1200
+Wire Wire Line
+	5000 1200 5300 1200
+Wire Wire Line
+	5300 1200 5300 1300
+Connection ~ 5000 1200
+Wire Wire Line
+	5000 1200 5000 1150
+Wire Wire Line
+	5000 1550 5000 1600
+Connection ~ 5000 1600
+Wire Wire Line
+	5000 1600 4350 1600
 $EndSCHEMATC

Commit message: added GPIO3 to the OnOff button via a diode to allow for the Pi to be turned on
Parts:
- added D?: 1N4148W, Diode_SMD:D_SOD-123, symbol Diode:1N4148W
Other:
- note added: "GPIO3 boots\nPi when pulled\ndown via On/Off\nbutton.\nDiode to avoid \nI2C triggering \nthe shutdown."
Changed lines of the file:
@@
 	2400 1200 1250 1200
 Wire Wire Line
-	1250 1300 2400 1300
-Wire Wire Line
 	1250 1400 2400 1400
-Wire Wire Line
-	2400 1600 1250 1600
 Wire Wire Line
 	1250 1700 2400 1700
@@
 Wire Wire Line
 	5000 1600 4350 1600
+$Comp
+L Diode:1N4148W D?
+U 1 1 5BC73CE0
+P 1100 1450
+F 0 "D?" V 1150 1650 50  0000 R CNN
+F 1 "1N4148W" V 1050 1900 50  0000 R CNN
+F 2 "Diode_SMD:D_SOD-123" H 1100 1275 50  0001 C CNN
+F 3 "https://www.vishay.com/docs/85748/1n4148w.pdf" H 1100 1450 50  0001 C CNN
+	1    1100 1450
+	0    -1   -1   0
+$EndComp
+Wire Wire Line
+	1100 1300 2400 1300
+Wire Wire Line
+	1100 1600 2400 1600
+Text Notes 550  2150 0    50   ~ 0
+GPIO3 boots\nPi when pulled\ndown via On/Off\nbutton.\nDiode to avoid \nI2C triggering \nthe shutdown.
 $EndSCHEMATC

Commit message: added header for serial and I2C
Parts:
- added J?: Conn_01x07_Male, Connector_PinHeader_2.54mm:PinHeader_1x07_P2.54mm_Vertical, symbol Connector:Conn_01x07_Male
Connections:
- wire segments 142 -> 152
Changed lines of the file:
@@
 Text Notes 550  2150 0    50   ~ 0
 GPIO3 boots\nPi when pulled\ndown via On/Off\nbutton.\nDiode to avoid \nI2C triggering \nthe shutdown.
+$Comp
+L Connector:Conn_01x07_Male J?
+U 1 1 5BC817D8
+P 5150 6900
+F 0 "J?" H 5256 7378 50  0000 C CNN
+F 1 "Conn_01x07_Male" H 5256 7287 50  0000 C CNN
+F 2 "Connector_PinHeader_2.54mm:PinHeader_1x07_P2.54mm_Vertical" H 5150 6900 50  0001 C CNN
+F 3 "~" H 5150 6900 50  0001 C CNN
+	1    5150 6900
+	1    0    0    -1
+$EndComp
+$Comp
+L power:GND #PWR?
+U 1 1 5BC81D19
+P 5400 7250
+F 0 "#PWR?" H 5400 7000 50  0001 C CNN
+F 1 "GND" H 5405 7077 50  0000 C CNN
+F 2 "" H 5400 7250 50  0001 C CNN
+F 3 "" H 5400 7250 50  0001 C CNN
+	1    5400 7250
+	1    0    0    -1
+$EndComp
+$Comp
+L power:+3.3V #PWR?
+U 1 1 5BC81DE1
+P 6050 6550
+F 0 "#PWR?" H 6050 6400 50  0001 C CNN
+F 1 "+3.3V" H 6065 6723 50  0000 C CNN
+F 2 "" H 6050 6550 50  0001 C CNN
+F 3 "" H 6050 6550 50  0001 C CNN
+	1    6050 6550
+	1    0    0    -1
+$EndComp
+$Comp
+L power:+5V #PWR?
+U 1 1 5BC81EB0
+P 5850 6550
+F 0 "#PWR?" H 5850 6400 50  0001 C CNN
+F 1 "+5V" H 5865 6723 50  0000 C CNN
+F 2 "" H 5850 6550 50  0001 C CNN
+F 3 "" H 5850 6550 50  0001 C CNN
+	1    5850 6550
+	1    0    0    -1
+$EndComp
+Wire Wire Line
+	5350 6600 5850 6600
+Wire Wire Line
+	5850 6600 5850 6550
+Wire Wire Line
+	5350 6700 6050 6700
+Wire Wire Line
+	6050 6700 6050 6550
+Wire Wire Line
+	5350 7200 5400 7200
+Wire Wire Line
+	5400 7200 5400 7250
+Wire Wire Line
+	5350 6800 6050 6800
+Wire Wire Line
+	5350 6900 6050 6900
+Wire Wire Line
+	5350 7000 6050 7000
+Wire Wire Line
+	5350 7100 6050 7100
+Text Label 6050 6800 2    50   ~ 0
+GPIO14(TXD0)
+Text Label 6050 6900 2    50   ~ 0
+GPIO15(RXD0)
+Text Label 6050 7000 2    50   ~ 0
+GPIO2(SDA1)
+Text Label 6050 7100 2    50   ~ 0
+GPIO3(SCL1)
 $EndSCHEMATC

Commit message: updated layout to the new changes
Parts:
- J3: renamed from J?; footprint Connector_PinHeader_2.54mm:PinHeader_1x07_P2.54mm_Vertical -> Connector_PinHeader_2.54mm:PinHeader_1x07_P2.54mm_Horizontal
- gave numbers to parts that had none: 4
Changed lines of the file:
@@
 	5800 1500 5800 1200
 $Comp
-L Transistor_FET:BSS138 Q?
+L Transistor_FET:BSS138 Q1
 U 1 1 5BBD252E
 P 5300 1500
-F 0 "Q?" V 5550 1500 50  0000 C CNN
+F 0 "Q1" V 5550 1500 50  0000 C CNN
 F 1 "BSS138" V 5641 1500 50  0000 C CNN
 F 2 "Package_TO_SOT_SMD:SOT-23" H 5500 1425 50  0001 L CIN
@@
 $EndComp
 $Comp
-L Device:R R?
+L Device:R R22
 U 1 1 5BC07184
 P 5550 1400
-F 0 "R?" H 5620 1446 50  0000 L CNN
+F 0 "R22" H 5620 1446 50  0000 L CNN
 F 1 "10k" H 5620 1355 50  0000 L CNN
 F 2 "Resistor_SMD:R_0805_2012Metric_Pad1.15x1.40mm_HandSolder" V 5480 1400 50  0001 C CNN
@@
 	5100 1600 5000 1600
 $Comp
-L Device:R R?
+L Device:R R1
 U 1 1 5BC3AC59
 P 5000 1400
-F 0 "R?" H 5070 1446 50  0000 L CNN
+F 0 "R1" H 5070 1446 50  0000 L CNN
 F 1 "10k" H 5070 1355 50  0000 L CNN
 F 2 "Resistor_SMD:R_0805_2012Metric_Pad1.15x1.40mm_HandSolder" V 4930 1400 50  0001 C CNN
@@
 $EndComp
 $Comp
-L power:+3.3V #PWR?
+L power:+3.3V #PWR0127
 U 1 1 5BC3ADA5
 P 5000 1150
-F 0 "#PWR?" H 5000 1000 50  0001 C CNN
+F 0 "#PWR0127" H 5000 1000 50  0001 C CNN
 F 1 "+3.3V" H 5000 1290 50  0000 C CNN
 F 2 "" H 5000 1150 50  0000 C CNN
@@
 	5000 1600 4350 1600
 $Comp
-L Diode:1N4148W D?
+L Diode:1N4148W D1
 U 1 1 5BC73CE0
 P 1100 1450
-F 0 "D?" V 1150 1650 50  0000 R CNN
+F 0 "D1" V 1150 1650 50  0000 R CNN
 F 1 "1N4148W" V 1050 1900 50  0000 R CNN
 F 2 "Diode_SMD:D_SOD-123" H 1100 1275 50  0001 C CNN
@@
 GPIO3 boots\nPi when pulled\ndown via On/Off\nbutton.\nDiode to avoid \nI2C triggering \nthe shutdown.
 $Comp
-L Connector:Conn_01x07_Male J?
+L Connector:Conn_01x07_Male J3
 U 1 1 5BC817D8
 P 5150 6900
-F 0 "J?" H 5256 7378 50  0000 C CNN
+F 0 "J3" H 5256 7378 50  0000 C CNN
 F 1 "Conn_01x07_Male" H 5256 7287 50  0000 C CNN
-F 2 "Connector_PinHeader_2.54mm:PinHeader_1x07_P2.54mm_Vertical" H 5150 6900 50  0001 C CNN
+F 2 "Connector_PinHeader_2.54mm:PinHeader_1x07_P2.54mm_Horizontal" H 5150 6900 50  0001 C CNN
 F 3 "~" H 5150 6900 50  0001 C CNN
 	1    5150 6900
@@
 $EndComp
 $Comp
-L power:GND #PWR?
+L power:GND #PWR0128
 U 1 1 5BC81D19
 P 5400 7250
-F 0 "#PWR?" H 5400 7000 50  0001 C CNN
+F 0 "#PWR0128" H 5400 7000 50  0001 C CNN
 F 1 "GND" H 5405 7077 50  0000 C CNN
 F 2 "" H 5400 7250 50  0001 C CNN
@@
 $EndComp
 $Comp
-L power:+3.3V #PWR?
+L power:+3.3V #PWR0129
 U 1 1 5BC81DE1
 P 6050 6550
-F 0 "#PWR?" H 6050 6400 50  0001 C CNN
+F 0 "#PWR0129" H 6050 6400 50  0001 C CNN
 F 1 "+3.3V" H 6065 6723 50  0000 C CNN
 F 2 "" H 6050 6550 50  0001 C CNN
@@
 $EndComp
 $Comp
-L power:+5V #PWR?
+L power:+5V #PWR0130
 U 1 1 5BC81EB0
 P 5850 6550
-F 0 "#PWR?" H 5850 6400 50  0001 C CNN
+F 0 "#PWR0130" H 5850 6400 50  0001 C CNN
 F 1 "+5V" H 5865 6723 50  0000 C CNN
 F 2 "" H 5850 6550 50  0001 C CNN
